File: Margay.brd (EAGLE design)
At the start: 50.2 x 30.4 mm, 61 parts, among them IC1 ATMEGA644M, J1 CONN_4SCREW_2.54, J2 CONN_6, Q1 MOSFET_PCH-IRLML2244, Q2 MOSFET-NCH-DMG3404L, Q5 MOSFET_PCH-IRLML2244, U2 FT231X-Q

Commit message: Final Gerbers, renamed design
Parts:
- JP2: value JUMPER-SMT_2_NO_SILK -> JUMPER-SMT_2_NC_PASTE_SILK; device SparkFun-Jumpers:SMT-JUMPER_2_NO_SILK -> SparkFun-Jumpers:SMT-JUMPER_2_NC_PASTE_SILK
Other:
- board text added: "Project Margay v0.0 ---------------- Developed by Northern Widget and University of Minnesota"
- board text removed: "Project Blackfoot v0.0 ---------------- Developed by Northern Widget and University of Minnesota"
Changed lines of the file:
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@@
 <layer number="29" name="tStop" color="7" fill="3" visible="no" active="yes"/>
 <layer number="30" name="bStop" color="7" fill="6" visible="no" active="yes"/>
-<layer number="31" name="tCream" color="7" fill="4" visible="no" active="yes"/>
+<layer number="31" name="tCream" color="7" fill="4" visible="yes" active="yes"/>
 <layer number="32" name="bCream" color="7" fill="5" visible="no" active="yes"/>
 <layer number="33" name="tFinish" color="6" fill="3" visible="no" active="yes"/>
@@
 <text x="13.716" y="28.829" size="0.8128" layer="51" font="vector" ratio="15" distance="40" rot="SR90" align="center">STAT</text>
 <text x="34.544" y="19.558" size="0.8128" layer="51" font="vector" ratio="15" distance="40" align="center">AUX</text>
-<text x="49.53" y="21.971" size="0.8128" layer="22" font="vector" ratio="15" distance="40" rot="MR0" align="center-left">Project Blackfoot v0.0
+<text x="49.53" y="21.971" size="0.8128" layer="22" font="vector" ratio="15" distance="40" rot="MR0" align="center-left">Project Margay v0.0
 ----------------
 Developed by
@@
 <element name="J5" library="bschulz" package="1X02_2.54_SCREWTERM" value="" x="46.355" y="5.969" rot="R270"/>
 <element name="JP1" library="SparkFun-Jumpers" library_urn="urn:adsk.eagle:library:528" package="SMT-JUMPER_3_1-NC_PASTE_SILK" package3d_urn="urn:adsk.eagle:package:39293/1" value="JUMPER-SMT_3_1-NC_PASTE_SILK" x="43.561" y="6.096" rot="MR270"/>
-<element name="JP2" library="SparkFun-Jumpers" library_urn="urn:adsk.eagle:library:528" package="SMT-JUMPER_2_NO_SILK" package3d_urn="urn:adsk.eagle:package:39279/1" value="JUMPER-SMT_2_NO_SILK" x="38.481" y="11.938"/>
+<element name="JP2" library="SparkFun-Jumpers" library_urn="urn:adsk.eagle:library:528" package="SMT-JUMPER_2_NC_PASTE_SILK" package3d_urn="urn:adsk.eagle:package:39282/1" value="JUMPER-SMT_2_NC_PASTE_SILK" x="38.481" y="11.938"/>
 <element name="MICRO_USB" library="bschulz" package="10118194-0001LF_10118194-0001LF_LONGER_PADS" value="MICRO_USB_LONGPADS" x="40.894" y="28.956" rot="R180"/>
 <element name="Q1" library="bschulz" package="SOT23-3" value="MOSFET_PCH-IRLML2244" x="41.148" y="4.318" rot="R90">
