File: Margay.sch (EAGLE design)
At the start: 60 parts, among them IC1 ATMEGA644M, J1 CONN_4SCREW_2.54, J2 CONN_6, Q1 MOSFET_PCH-IRLML2244, Q2 MOSFET-NCH-DMG3404L, Q5 MOSFET_PCH-IRLML2244, U2 FT231X-Q

Commit message: Final Gerbers, renamed design
Parts:
- JP2: value JUMPER-SMT_2_NO_SILK -> JUMPER-SMT_2_NC_PASTE_SILK; device SparkFun-Jumpers:JUMPER-SMT_2_NO_SILK -> SparkFun-Jumpers:JUMPER-SMT_2_NC_PASTE_SILK
Changed lines of the file:
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@@
 <part name="J5" library="bschulz" deviceset="CONN_02" device="2.54MM_SCREWTERM"/>
 <part name="R12" library="bschulz" deviceset="R-EU_" device="R0603" value="10k"/>
-<part name="JP2" library="SparkFun-Jumpers" library_urn="urn:adsk.eagle:library:528" deviceset="JUMPER-SMT_2_NO" device="_SILK" package3d_urn="urn:adsk.eagle:package:39279/1"/>
+<part name="JP2" library="SparkFun-Jumpers" library_urn="urn:adsk.eagle:library:528" deviceset="JUMPER-SMT_2_NC_PASTE" device="_SILK" package3d_urn="urn:adsk.eagle:package:39282/1"/>
 <part name="R15" library="bschulz" deviceset="R-EU_" device="R0603" value="10k"/>
 <part name="GND8" library="supply1" library_urn="urn:adsk.eagle:library:371" deviceset="GND" device=""/>
