File: Hardware/KiCAD/Margay_3.kicad_sch (KiCad schematic)
At the start: 34 parts, among them Q1 MOSFET-NCH-DMG3404L, Q2 MOSFET_PCH-FDN360P, Q3 MOSFET-NCH-2N7002PW, U10 TLV3691DPF, U11 MIC9409C6, U12 BME280, U13 MAX6070AAUT, U14 MCP342, U6 TPS797, U7 TPS7A05DBV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

Commit message: 3V3 --> Schottky diode --> VCoin+. Provide a backup option for the clock if its battery fails: the main batteries of the data logger. Ideally, this would have been connected to VBat to keep the coin cell as just a backup. But I cannot see how to route that trace. However, this will at least serve to protect timekeeping.
Parts:
- added D4: BAT43WS, Margay:SOD323-R, symbol Margay-eagle-import:DIODESOD-323
Connections:
- net 3V3: now also D4.A
- net at BT1.POWER0 (+), BT1.POWER1 (+), C19.1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: now also D4.C
Changed lines of the file:
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@@
   (junction (at 40.64 180.34) (diameter 0) (color 0 0 0 0)
   )
+  (junction (at 266.7 172.72) (diameter 0) (color 0 0 0 0)
+  )
   (junction (at 50.8 48.26) (diameter 0) (color 0 0 0 0)
   )
@@
     (stroke (width 0.1524) (type solid))
   )
+  (wire (pts (xy 266.7 156.21) (xy 266.7 161.29))
+    (stroke (width 0) (type default))
+  )
   (wire (pts (xy 119.38 81.28) (xy 119.38 78.74))
     (stroke (width 0.1524) (type solid))
@@
     (stroke (width 0.1524) (type solid))
   )
+  (wire (pts (xy 266.7 166.37) (xy 266.7 172.72))
+    (stroke (width 0) (type default))
+  )
   (wire (pts (xy 248.92 170.18) (xy 251.46 170.18))
     (stroke (width 0.1524) (type solid))
@@
   (wire (pts (xy 177.8 63.5) (xy 177.8 66.04))
     (stroke (width 0.1524) (type solid))
+  )
+  (wire (pts (xy 266.7 156.21) (xy 270.51 156.21))
+    (stroke (width 0) (type default))
   )
   (wire (pts (xy 68.58 213.36) (xy 66.04 213.36))
@@
     (effects (font (size 0.889 0.889)) (justify left))
     (property "Intersheetrefs" "${INTERSHEET_REFS}" (at 266.6463 63.5 0)
+      (effects (font (size 1.27 1.27)) (justify left) hide)
+    )
+  )
+  (global_label "3V3" (shape bidirectional) (at 270.51 156.21 0) (fields_autoplaced)
+    (effects (font (size 0.889 0.889)) (justify left))
+    (property "Intersheetrefs" "${INTERSHEET_REFS}" (at 275.8328 156.21 0)
       (effects (font (size 1.27 1.27)) (justify left) hide)
     )
@@
         )
       )
+    )
+  )
+  (symbol (lib_id "Margay-eagle-import:DIODESOD-323") (at 266.7 163.83 270) (unit 1)
+    (in_bom yes) (on_board yes) (dnp no)
+    (property "Reference" "D4" (at 267.1826 166.37 0)
+      (effects (font (size 1.778 1.5113)) (justify left bottom))
+    )
+    (property "Value" "BAT43WS" (at 261.8486 161.29 0)
+      (effects (font (size 1.778 1.5113)) (justify left bottom))
+    )
+    (property "Footprint" "Margay:SOD323-R" (at 266.7 163.83 0)
+      (effects (font (size 1.27 1.27)) hide)
+    )
+    (property "Datasheet" "" (at 266.7 163.83 0)
+      (effects (font (size 1.27 1.27)) hide)
+    )
+    (property "DIGIKEY" "BAT43WS-FDICT-ND" (at 266.7 163.83 0)
+      (effects (font (size 1.27 1.27)) hide)
+    )
+    (property "MF" "Diodes Incorporated" (at 266.7 163.83 0)
+      (effects (font (size 1.27 1.27)) hide)
+    )
+    (property "MPN" "BAT43WS-7-F" (at 266.7 163.83 0)
+      (effects (font (size 1.27 1.27)) hide)
+    )
+    (pin "A")
+    (pin "C")
+    (instances
+      (project "Margay"
+        (path "/44591453-0fe4-48d8-a9e2-921075afaa78/8b29bb9a-8b12-402b-8332-650c6f7ae85e"
+          (reference "D4") (unit 1)
+        )
+      )

Commit message: Add extra 1 uA decoupling cap for DS3231M. The 0.1uF cap is right by the battery, which is fine. But there was not as much buffering of power changes right by the DS3231M. And the DS3231M responds better the closer the capacitor is.
Claude Code did a quick calculation based on my finding of an up to 300 us
lag: this is the time required for a VBat handoff.
C = I × t / ΔV = 0.3 mA × 300 µs / 0.25 V = 0.36 µF

This extra capacitor might not be necessary, but considering the importance
of the RTC and the fact that we have space, I am aiming these commits to
ensure that the RTC is properly buffered from power changes and stays running.
Parts:
- added C20: 1uF, Margay:C0603, symbol Margay-eagle-import:C-EUC0603
Connections:
- net GND: now also C20.2
- net at BT1.POWER0 (+), BT1.POWER1 (+), C19.1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: now also C20.1
Changed lines of the file:
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@@
   (junction (at 246.38 139.7) (diameter 0) (color 0 0 0 0)
   )
+  (junction (at 266.7 180.34) (diameter 0) (color 0 0 0 0)
+  )
   (wire (pts (xy 53.34 58.42) (xy 58.42 58.42))
     (stroke (width 0.1524) (type solid))
@@
   )
   (wire (pts (xy 96.52 205.74) (xy 99.06 205.74))
+    (stroke (width 0.1524) (type solid))
+  )
+  (wire (pts (xy 266.7 172.72) (xy 279.4 172.72))
     (stroke (width 0.1524) (type solid))
   )
@@
   )
   (wire (pts (xy 218.44 129.54) (xy 215.9 129.54))
+    (stroke (width 0.1524) (type solid))
+  )
+  (wire (pts (xy 266.7 180.34) (xy 279.4 180.34))
     (stroke (width 0.1524) (type solid))
   )
@@
   (symbol (lib_id "Margay-eagle-import:GND") (at 259.08 185.42 0) (unit 1)
     (in_bom yes) (on_board yes) (dnp no)
-    (property "Reference" "#GND32" (at 259.08 185.42 0)
+    (property "Reference" "#GND032" (at 259.08 185.42 0)
       (effects (font (size 1.27 1.27)) hide)
     )
@@
       (project "Margay"
         (path "/44591453-0fe4-48d8-a9e2-921075afaa78/8b29bb9a-8b12-402b-8332-650c6f7ae85e"
-          (reference "#GND32") (unit 1)
+          (reference "#GND032") (unit 1)
         )
       )
@@
   (symbol (lib_id "Margay-eagle-import:SparkFun-PowerSymbols_GND") (at 63.5 83.82 0) (unit 1)
     (in_bom yes) (on_board yes) (dnp no)
-    (property "Reference" "#GND20" (at 63.5 83.82 0)
+    (property "Reference" "#GND020" (at 63.5 83.82 0)
       (effects (font (size 1.27 1.27)) hide)
     )
@@
       (project "Margay"
         (path "/44591453-0fe4-48d8-a9e2-921075afaa78/8b29bb9a-8b12-402b-8332-650c6f7ae85e"
-          (reference "#GND20") (unit 1)
+          (reference "#GND020") (unit 1)
         )
       )
@@
   (symbol (lib_id "Margay-eagle-import:GND") (at 248.92 111.76 0) (unit 1)
     (in_bom yes) (on_board yes) (dnp no)
-    (property "Reference" "#GND30" (at 248.92 111.76 0)
+    (property "Reference" "#GND030" (at 248.92 111.76 0)
       (effects (font (size 1.27 1.27)) hide)
     )
@@
       (project "Margay"
         (path "/44591453-0fe4-48d8-a9e2-921075afaa78/8b29bb9a-8b12-402b-8332-650c6f7ae85e"
-          (reference "#GND30") (unit 1)
+          (reference "#GND030") (unit 1)
         )
       )
@@
   (symbol (lib_id "Margay-eagle-import:GND") (at 177.8 68.58 0) (unit 1)
     (in_bom yes) (on_board yes) (dnp no)
-    (property "Reference" "#GND26" (at 177.8 68.58 0)
+    (property "Reference" "#GND026" (at 177.8 68.58 0)
       (effects (font (size 1.27 1.27)) hide)
     )
@@
       (project "Margay"
         (path "/44591453-0fe4-48d8-a9e2-921075afaa78/8b29bb9a-8b12-402b-8332-650c6f7ae85e"
-          (reference "#GND26") (unit 1)
+          (reference "#GND026") (unit 1)
         )
       )
@@
   (symbol (lib_id "Margay-eagle-import:GND") (at 40.64 195.58 0) (unit 1)
     (in_bom yes) (on_board yes) (dnp no)
-    (property "Reference" "#GND18" (at 40.64 195.58 0)
+    (property "Reference" "#GND018" (at 40.64 195.58 0)
       (effects (font (size 1.27 1.27)) hide)
     )
@@
       (project "Margay"
         (path "/44591453-0fe4-48d8-a9e2-921075afaa78/8b29bb9a-8b12-402b-8332-650c6f7ae85e"
-          (reference "#GND18") (unit 1)
+          (reference "#GND018") (unit 1)
         )
       )
@@
   (symbol (lib_id "Margay-eagle-import:GND") (at 251.46 187.96 0) (unit 1)
     (in_bom yes) (on_board yes) (dnp no)
-    (property "Reference" "#GND31" (at 251.46 187.96 0)
+    (property "Reference" "#GND031" (at 251.46 187.96 0)
       (effects (font (size 1.27 1.27)) hide)
     )
@@
       (project "Margay"
         (path "/44591453-0fe4-48d8-a9e2-921075afaa78/8b29bb9a-8b12-402b-8332-650c6f7ae85e"
-          (reference "#GND31") (unit 1)
+          (reference "#GND031") (unit 1)
         )
       )
@@
   (symbol (lib_id "Margay-eagle-import:GND") (at 58.42 60.96 0) (unit 1)
     (in_bom yes) (on_board yes) (dnp no)
-    (property "Reference" "#GND19" (at 58.42 60.96 0)
+    (property "Reference" "#GND019" (at 58.42 60.96 0)
       (effects (font (size 1.27 1.27)) hide)
     )
@@
       (project "Margay"
         (path "/44591453-0fe4-48d8-a9e2-921075afaa78/8b29bb9a-8b12-402b-8332-650c6f7ae85e"
-          (reference "#GND19") (unit 1)
+          (reference "#GND019") (unit 1)
         )
       )
@@
   (symbol (lib_id "Margay-eagle-import:GND") (at 254 78.74 0) (unit 1)
     (in_bom yes) (on_board yes) (dnp no)
-    (property "Reference" "#GND28" (at 254 78.74 0)
+    (property "Reference" "#GND028" (at 254 78.74 0)
       (effects (font (size 1.27 1.27)) hide)
     )
@@
       (project "Margay"
         (path "/44591453-0fe4-48d8-a9e2-921075afaa78/8b29bb9a-8b12-402b-8332-650c6f7ae85e"
-          (reference "#GND28") (unit 1)
+          (reference "#GND028") (unit 1)
         )
       )
@@
   (symbol (lib_id "Margay-eagle-import:GND") (at 109.22 60.96 0) (unit 1)
     (in_bom yes) (on_board yes) (dnp no)
-    (property "Reference" "#GND24" (at 109.22 60.96 0)
+    (property "Reference" "#GND024" (at 109.22 60.96 0)
       (effects (font (size 1.27 1.27)) hide)
     )
@@
       (project "Margay"
         (path "/44591453-0fe4-48d8-a9e2-921075afaa78/8b29bb9a-8b12-402b-8332-650c6f7ae85e"
-          (reference "#GND24") (unit 1)
+          (reference "#GND024") (unit 1)
         )
       )
@@
   (symbol (lib_id "Margay-eagle-import:GND") (at 99.06 210.82 0) (unit 1)
     (in_bom yes) (on_board yes) (dnp no)
-    (property "Reference" "#GND23" (at 99.06 210.82 0)
+    (property "Reference" "#GND023" (at 99.06 210.82 0)
       (effects (font (size 1.27 1.27)) hide)
     )
@@
       (project "Margay"
         (path "/44591453-0fe4-48d8-a9e2-921075afaa78/8b29bb9a-8b12-402b-8332-650c6f7ae85e"
-          (reference "#GND23") (unit 1)
+          (reference "#GND023") (unit 1)
         )
       )
@@
   (symbol (lib_id "Margay-eagle-import:GND") (at 246.38 144.78 0) (unit 1)
     (in_bom yes) (on_board yes) (dnp no)
-    (property "Reference" "#GND29" (at 246.38 144.78 0)
+    (property "Reference" "#GND029" (at 246.38 144.78 0)
       (effects (font (size 1.27 1.27)) hide)
     )
@@
       (project "Margay"
         (path "/44591453-0fe4-48d8-a9e2-921075afaa78/8b29bb9a-8b12-402b-8332-650c6f7ae85e"
-          (reference "#GND29") (unit 1)
+          (reference "#GND029") (unit 1)
         )
       )
@@
   (symbol (lib_id "Margay-eagle-import:GND") (at 208.28 147.32 0) (unit 1)
     (in_bom yes) (on_board yes) (dnp no)
-    (property "Reference" "#GND27" (at 208.28 147.32 0)
+    (property "Reference" "#GND027" (at 208.28 147.32 0)
       (effects (font (size 1.27 1.27)) hide)
     )
@@
       (project "Margay"
         (path "/44591453-0fe4-48d8-a9e2-921075afaa78/8b29bb9a-8b12-402b-8332-650c6f7ae85e"
-          (reference "#GND27") (unit 1)
+          (reference "#GND027") (unit 1)
         )
       )
@@
   (symbol (lib_id "Margay-eagle-import:SparkFun-PowerSymbols_GND") (at 119.38 83.82 0) (unit 1)
     (in_bom yes) (on_board yes) (dnp no)
-    (property "Reference" "#GND25" (at 119.38 83.82 0)
+    (property "Reference" "#GND025" (at 119.38 83.82 0)
       (effects (font (size 1.27 1.27)) hide)
     )
@@
       (project "Margay"
         (path "/44591453-0fe4-48d8-a9e2-921075afaa78/8b29bb9a-8b12-402b-8332-650c6f7ae85e"
-          (reference "#GND25") (unit 1)
+          (reference "#GND025") (unit 1)
         )
       )
@@
     )
   )
+  (symbol (lib_id "Margay-eagle-import:C-EUC0603") (at 279.4 175.26 0) (unit 1)
+    (in_bom yes) (on_board yes) (dnp no)
+    (property "Reference" "C20" (at 280.924 174.879 0)
+      (effects (font (size 1.778 1.5113)) (justify left bottom))
+    )
+    (property "Value" "1uF" (at 280.924 179.959 0)
+      (effects (font (size 1.778 1.5113)) (justify left bottom))
+    )
+    (property "Footprint" "Margay:C0603" (at 279.4 175.26 0)
+      (effects (font (size 1.27 1.27)) hide)
+    )
+    (property "Datasheet" "" (at 279.4 175.26 0)
+      (effects (font (size 1.27 1.27)) hide)
+    )
+    (pin "1")
+    (pin "2")
+    (instances
+      (project "Margay"
+        (path "/44591453-0fe4-48d8-a9e2-921075afaa78/8b29bb9a-8b12-402b-8332-650c6f7ae85e"
+          (reference "C20") (unit 1)
+        )
+      )
+    )
+  )
   (symbol (lib_id "Margay-eagle-import:C-EUC0402") (at 208.28 137.16 0) (unit 1)
     (in_bom yes) (on_board yes) (dnp no)
@@
   (symbol (lib_id "Margay-eagle-import:SparkFun-PowerSymbols_GND") (at 93.98 121.92 0) (unit 1)
     (in_bom yes) (on_board yes) (dnp no)
-    (property "Reference" "#GND22" (at 93.98 121.92 0)
+    (property "Reference" "#GND022" (at 93.98 121.92 0)
       (effects (font (size 1.27 1.27)) hide)
     )
@@
       (project "Margay"
         (path "/44591453-0fe4-48d8-a9e2-921075afaa78/8b29bb9a-8b12-402b-8332-650c6f7ae85e"
-          (reference "#GND22") (unit 1)
+          (reference "#GND022") (unit 1)
         )
       )
@@
   (symbol (lib_id "Margay-eagle-import:GND") (at 68.58 165.1 0) (unit 1)
     (in_bom yes) (on_board yes) (dnp no)
-    (property "Reference" "#GND21" (at 68.58 165.1 0)
+    (property "Reference" "#GND021" (at 68.58 165.1 0)
       (effects (font (size 1.27 1.27)) hide)
     )
@@
       (project "Margay"
         (path "/44591453-0fe4-48d8-a9e2-921075afaa78/8b29bb9a-8b12-402b-8332-650c6f7ae85e"
-          (reference "#GND21") (unit 1)
-        )
-      )
+          (reference "#GND021") (unit 1)
+        )
+      )

Commit message: Unify 10K resistors to CRT0603-BY-1002ELFCT-ND.
Parts:
- R22: DIGIKEY (none) -> CRT0603-BY-1002ELFCT-ND; MF (none) -> Bourns; MPN (none) -> CRT0603-BY-1002ELF
- R23: DIGIKEY (none) -> CRT0603-BY-1002ELFCT-ND; MF (none) -> Bourns; MPN (none) -> CRT0603-BY-1002ELFCT-ND
Changed lines of the file:
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@@
+      (effects (font (size 1.27 1.27)) hide)
+    )
+    (property "DIGIKEY" "CRT0603-BY-1002ELFCT-ND" (at 254 55.88 0)
+      (effects (font (size 1.27 1.27)) hide)
+    )
+    (property "MF" "Bourns" (at 254 55.88 0)
+      (effects (font (size 1.27 1.27)) hide)
+    )
+    (property "MPN" "CRT0603-BY-1002ELF" (at 254 55.88 0)
       (effects (font (size 1.27 1.27)) hide)
     )
@@
       (effects (font (size 1.27 1.27)) hide)
     )
+    (property "DIGIKEY" "CRT0603-BY-1002ELFCT-ND" (at 254 68.58 0)
+      (effects (font (size 1.27 1.27)) hide)
+    )
+    (property "MF" "Bourns" (at 254 68.58 0)
+      (effects (font (size 1.27 1.27)) hide)
+    )
+    (property "MPN" "CRT0603-BY-1002ELFCT-ND" (at 254 68.58 0)
+      (effects (font (size 1.27 1.27)) hide)
+    )
