File: Hardware/KiCAD/Margay_3.kicad_sch (KiCad schematic)
At the start: 36 parts, among them Q1 MOSFET-NCH-DMG3404L, Q2 MOSFET_PCH-FDN360P, Q3 MOSFET-NCH-2N7002PW, U10 TLV3691DPF, U11 MIC9409C6, U12 BME280, U13 MAX6070AAUT, U14 MCP342, U6 TPS797, U7 TPS7A05DBV, U8 TPS22916YFP, U9 TPS210

Commit message: KiCAD: populate MPN/MF/DIGIKEY fields from v3.0 BoM CSV
72 components updated with manufacturer, MPN, and DigiKey fields from
Margay_BoM_3v0_-_2023-03-17.csv. Fields were absent after Eagle→KiCAD
import. C20 (new 1µF DS3231M VCC decoupling cap) assigned same part as
C13/C14 (TMK107B7105KA-T). R22/R23 preserved as CRT0603-BY-1002ELF
(already correct). R7/R9 skipped — BoM MPN is a 330Ω part number, wrong
for the 1k value; needs manual correction.

Co-Authored-By: Claude Sonnet 4.6 <noreply@anthropic.com>
Parts:
- BT1: DIGIKEY (none) -> BAT-HLD-012-SMT-ND; MF (none) -> Linx; MPN (none) -> BAT-HLD-012-SMT
- C10, C11, C12, C16, C17, C18, C19: DIGIKEY (none) -> 490-4759-1-ND; MF (none) -> Murata; MPN (none) -> GCM155R71C104KA55D
- C13, C14, C20: DIGIKEY (none) -> 587-2984-1-ND; MF (none) -> Yaiyo Yuden; MPN (none) -> TMK107B7105KA-T
- C15: DIGIKEY (none) -> 490-6473-1-ND; MF (none) -> Murata; MPN (none) -> GRM21BR61C106KE15K
- JP2, JP3: DIGIKEY (none) -> DNP; MF (none) -> N/A; MPN (none) -> N/A
- Q1: DIGIKEY (none) -> DMG3404L-7DICT-ND; MF (none) -> Diodes Incorporated; MPN (none) -> DMG3404L-7
- Q3: DIGIKEY (none) -> 2N7002W-FDICT-ND; MF (none) -> Diodes Incorporated; MPN (none) -> 2N7002W-7-F
- R17, R18, R20, R21: DIGIKEY (none) -> 311-10.0KLRCT-ND; MF (none) -> Yageo; MPN (none) -> RC0402FR-0710KL
- R19: DIGIKEY (none) -> 311-100LRCT-ND; MF (none) -> Yageo; MPN (none) -> RC0402FR-07100RL
- RTC1: DIGIKEY (none) -> DS3231MZ+-ND; MF (none) -> Maxim; MPN (none) -> DS3231MZ+
- U10: DIGIKEY (none) -> 296-37242-6-ND; MF (none) -> TI; MPN (none) -> TLV3691IDPFR
- U11: DIGIKEY (none) -> 576-3484-1-ND; MF (none) -> Microchip; MPN (none) -> MIC94090YC6-TR
- U12: DIGIKEY (none) -> 828-1063-1-ND; MF (none) -> Bosch; MPN (none) -> BME280
- U13: DIGIKEY MAX6070AAUT18+TCT-ND -> MAX6070BAUT18+TCT-ND; MF (none) -> Maxim; MPN MAX6071AAUT18+T -> MAX6070BAUT18+T
- U14: DIGIKEY (none) -> MCP3421A1T-E/CHCT-ND; MF (none) -> Microchip; MPN (none) -> MCP3421A1T-E/CH
- U6: DIGIKEY (none) -> 296-11990-1-ND; MF (none) -> TI; MPN (none) -> TPS79733DCKR
- U7: DIGIKEY (none) -> 296-50256-1-ND; MF (none) -> TI; MPN (none) -> TPS7A0533PDBVR
- U8: DIGIKEY (none) -> 296-47464-1-ND; MF (none) -> TI; MPN (none) -> TPS22916CYFPT
- U9: MF (none) -> TI
