File: Hardware/KiCAD/Margay_2.kicad_sch (KiCad schematic)
At the start: 19 parts, among them J2 CONN_102.54_SCREW, J3 CONN_6SCREW_2.54, U3 TPL5010DDC, U4 SN74LVC1G3157SC70, U5 SN74AUP3G34DCU

Commit message: KiCAD: populate MPN/MF/DIGIKEY fields from v3.0 BoM CSV
72 components updated with manufacturer, MPN, and DigiKey fields from
Margay_BoM_3v0_-_2023-03-17.csv. Fields were absent after Eagle→KiCAD
import. C20 (new 1µF DS3231M VCC decoupling cap) assigned same part as
C13/C14 (TMK107B7105KA-T). R22/R23 preserved as CRT0603-BY-1002ELF
(already correct). R7/R9 skipped — BoM MPN is a 330Ω part number, wrong
for the 1k value; needs manual correction.

Co-Authored-By: Claude Sonnet 4.6 <noreply@anthropic.com>
Parts:
- D2, D3: DIGIKEY (none) -> CLVBA-FKA-CAEDH8BBB7A363CT-ND; MF (none) -> Cree; MPN (none) -> CLVBA-FKA-CAEDH8BBB7A363
- J2: DIGIKEY (none) -> ED10567-ND; MF (none) -> On Shore; MPN (none) -> OSTVN10A150
- J3: DIGIKEY (none) -> ED10565-ND; MF (none) -> OnShore; MPN (none) -> OSTVN06A150
- JP1: DIGIKEY (none) -> DNP; MF (none) -> N/A; MPN (none) -> N/A
- R10: DIGIKEY (none) -> 311-130KHRCT-ND; MF (none) -> Yageo; MPN (none) -> RC0603FR-07130KL
- R11, R12, R13, R5, R6: DIGIKEY (none) -> 311-330LRCT-ND; MF (none) -> Yageo; MPN (none) -> RC0402FR-07330RL
- R14: DIGIKEY (none) -> 311-10.0KLRCT-ND; MF (none) -> Yageo; MPN (none) -> RC0402FR-0710KL
- R8: DIGIKEY (none) -> 311-330LRCT-ND; MPN (none) -> RC0402FR-07330RL
- S1, S2: DIGIKEY (none) -> CKN10504CT-ND; MF (none) -> C&K; MPN (none) -> PTS810 SJG 250 SMTR LFS
- U3: DIGIKEY (none) -> 296-38829-1-ND; MF (none) -> TI; MPN (none) -> TPL5010DDCT
- U4: DIGIKEY (none) -> 296-14909-1-ND; MF (none) -> TI; MPN (none) -> SN74LVC1G3157DCKR
- U5: DIGIKEY (none) -> 296-25595-1-ND; MF (none) -> TI; MPN (none) -> SN74AUP3G34DCUR
Changed lines of the file:
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@@
+      (effects (font (size 1.27 1.27)) hide)
+    )
+    (property "MPN" "SN74LVC1G3157DCKR" (at 226.06 111.76 0)
+      (effects (font (size 1.27 1.27)) hide)
+    )
+    (property "MF" "TI" (at 226.06 111.76 0)
+      (effects (font (size 1.27 1.27)) hide)
+    )
+    (property "DIGIKEY" "296-14909-1-ND" (at 226.06 111.76 0)
       (effects (font (size 1.27 1.27)) hide)
     )
@@
       (effects (font (size 1.27 1.27)) hide)
     )
+    (property "MPN" "RC0402FR-07330RL" (at 58.42 101.6 0)
+      (effects (font (size 1.27 1.27)) hide)
+    )
+    (property "MF" "Yageo" (at 58.42 101.6 0)
+      (effects (font (size 1.27 1.27)) hide)
+    )
+    (property "DIGIKEY" "311-330LRCT-ND" (at 58.42 101.6 0)
+      (effects (font (size 1.27 1.27)) hide)
+    )
     (pin "1")
     (pin "2")
@@
       (effects (font (size 1.27 1.27)) hide)
     )
+    (property "MPN" "PTS810 SJG 250 SMTR LFS" (at 137.16 210.82 0)
+      (effects (font (size 1.27 1.27)) hide)
+    )
+    (property "MF" "C&K" (at 137.16 210.82 0)
+      (effects (font (size 1.27 1.27)) hide)
+    )
+    (property "DIGIKEY" "CKN10504CT-ND" (at 137.16 210.82 0)
+      (effects (font (size 1.27 1.27)) hide)
+    )
     (pin "1")
     (pin "2")
@@
       (effects (font (size 1.27 1.27)) hide)
     )
+    (property "MPN" "CLVBA-FKA-CAEDH8BBB7A363" (at 99.568 86.36 0)
+      (effects (font (size 1.27 1.27)) hide)
+    )
+    (property "MF" "Cree" (at 99.568 86.36 0)
+      (effects (font (size 1.27 1.27)) hide)
+    )
+    (property "DIGIKEY" "CLVBA-FKA-CAEDH8BBB7A363CT-ND" (at 99.568 86.36 0)
+      (effects (font (size 1.27 1.27)) hide)
+    )
     (pin "1")
     (pin "2")
@@
     )
     (property "Datasheet" "" (at 73.66 101.6 0)
+      (effects (font (size 1.27 1.27)) hide)
+    )
+    (property "MPN" "RC0402FR-07330RL" (at 73.66 101.6 0)
+      (effects (font (size 1.27 1.27)) hide)
+    )
+    (property "MF" "Yageo" (at 73.66 101.6 0)
+      (effects (font (size 1.27 1.27)) hide)
+    )
+    (property "DIGIKEY" "311-330LRCT-ND" (at 73.66 101.6 0)
       (effects (font (size 1.27 1.27)) hide)
     )
@@
       (effects (font (size 1.27 1.27)) hide)
     )
+    (property "MPN" "PTS810 SJG 250 SMTR LFS" (at 137.16 198.12 0)
+      (effects (font (size 1.27 1.27)) hide)
+    )
+    (property "MF" "C&K" (at 137.16 198.12 0)
+      (effects (font (size 1.27 1.27)) hide)
+    )
+    (property "DIGIKEY" "CKN10504CT-ND" (at 137.16 198.12 0)
+      (effects (font (size 1.27 1.27)) hide)
+    )
     (pin "4")
     (pin "3")
@@
     )
     (property "Datasheet" "" (at 48.26 218.44 0)
+      (effects (font (size 1.27 1.27)) hide)
+    )
+    (property "MPN" "OSTVN10A150" (at 48.26 218.44 0)
+      (effects (font (size 1.27 1.27)) hide)
+    )
+    (property "MF" "On Shore" (at 48.26 218.44 0)
+      (effects (font (size 1.27 1.27)) hide)
+    )
+    (property "DIGIKEY" "ED10567-ND" (at 48.26 218.44 0)
       (effects (font (size 1.27 1.27)) hide)
     )
@@
       (effects (font (size 1.27 1.27)) hide)
     )
+    (property "MPN" "TPL5010DDCT" (at 226.06 55.88 0)
+      (effects (font (size 1.27 1.27)) hide)
+    )
+    (property "MF" "TI" (at 226.06 55.88 0)
+      (effects (font (size 1.27 1.27)) hide)
+    )
+    (property "DIGIKEY" "296-38829-1-ND" (at 226.06 55.88 0)
+      (effects (font (size 1.27 1.27)) hide)
+    )
     (pin "1")
     (pin "2")
@@
       (effects (font (size 1.27 1.27)) hide)
     )
+    (property "MPN" "OSTVN06A150" (at 86.36 218.44 0)
+      (effects (font (size 1.27 1.27)) hide)
+    )
+    (property "MF" "OnShore" (at 86.36 218.44 0)
+      (effects (font (size 1.27 1.27)) hide)
+    )
+    (property "DIGIKEY" "ED10565-ND" (at 86.36 218.44 0)
+      (effects (font (size 1.27 1.27)) hide)
+    )
     (pin "1")
     (pin "2")
@@
       (effects (font (size 1.27 1.27)) hide)
     )
+    (property "MPN" "RC0402FR-07330RL" (at 91.694 101.6 0)
+      (effects (font (size 1.27 1.27)) hide)
+    )
+    (property "DIGIKEY" "311-330LRCT-ND" (at 91.694 101.6 0)
+      (effects (font (size 1.27 1.27)) hide)
+    )
     (property "MF" "Yageo" (at 91.694 101.6 0)
       (effects (font (size 1.27 1.27)) (justify left bottom) hide)
@@
     )
     (property "Datasheet" "" (at 226.06 86.36 0)
+      (effects (font (size 1.27 1.27)) hide)
+    )
+    (property "MPN" "SN74AUP3G34DCUR" (at 226.06 86.36 0)
+      (effects (font (size 1.27 1.27)) hide)
+    )
+    (property "MF" "TI" (at 226.06 86.36 0)
+      (effects (font (size 1.27 1.27)) hide)
+    )
+    (property "DIGIKEY" "296-25595-1-ND" (at 226.06 86.36 0)
       (effects (font (size 1.27 1.27)) hide)
     )
@@
       (effects (font (size 1.27 1.27)) hide)
     )
+    (property "MPN" "RC0402FR-07330RL" (at 106.68 101.6 0)
+      (effects (font (size 1.27 1.27)) hide)
+    )
+    (property "MF" "Yageo" (at 106.68 101.6 0)
+      (effects (font (size 1.27 1.27)) hide)
+    )
+    (property "DIGIKEY" "311-330LRCT-ND" (at 106.68 101.6 0)
+      (effects (font (size 1.27 1.27)) hide)
+    )
     (pin "1")
     (pin "2")
@@
     )
     (property "Datasheet" "" (at 99.568 101.6 0)
+      (effects (font (size 1.27 1.27)) hide)
+    )
+    (property "MPN" "RC0402FR-07330RL" (at 99.568 101.6 0)
+      (effects (font (size 1.27 1.27)) hide)
+    )
+    (property "MF" "Yageo" (at 99.568 101.6 0)
+      (effects (font (size 1.27 1.27)) hide)
+    )
+    (property "DIGIKEY" "311-330LRCT-ND" (at 99.568 101.6 0)
       (effects (font (size 1.27 1.27)) hide)
     )
@@
       (effects (font (size 1.27 1.27)) hide)
     )
+    (property "MPN" "CLVBA-FKA-CAEDH8BBB7A363" (at 66.04 86.36 0)
+      (effects (font (size 1.27 1.27)) hide)
+    )
+    (property "MF" "Cree" (at 66.04 86.36 0)
+      (effects (font (size 1.27 1.27)) hide)
+    )
+    (property "DIGIKEY" "CLVBA-FKA-CAEDH8BBB7A363CT-ND" (at 66.04 86.36 0)
+      (effects (font (size 1.27 1.27)) hide)
+    )
     (pin "1")
     (pin "2")
@@
     )
     (property "Datasheet" "" (at 200.66 60.96 0)
+      (effects (font (size 1.27 1.27)) hide)
+    )
+    (property "MPN" "RC0603FR-07130KL" (at 200.66 60.96 0)
+      (effects (font (size 1.27 1.27)) hide)
+    )
+    (property "MF" "Yageo" (at 200.66 60.96 0)
+      (effects (font (size 1.27 1.27)) hide)
+    )
+    (property "DIGIKEY" "311-130KHRCT-ND" (at 200.66 60.96 0)
       (effects (font (size 1.27 1.27)) hide)
     )
@@
       (effects (font (size 1.27 1.27)) hide)
     )
+    (property "MPN" "N/A" (at 147.32 172.72 0)
+      (effects (font (size 1.27 1.27)) hide)
+    )
+    (property "MF" "N/A" (at 147.32 172.72 0)
+      (effects (font (size 1.27 1.27)) hide)
+    )
+    (property "DIGIKEY" "DNP" (at 147.32 172.72 0)
+      (effects (font (size 1.27 1.27)) hide)
+    )
     (pin "1")
     (pin "2")
@@
       (effects (font (size 1.27 1.27)) hide)
     )
+    (property "MPN" "RC0402FR-0710KL" (at 157.48 195.58 0)
+      (effects (font (size 1.27 1.27)) hide)
+    )
+    (property "MF" "Yageo" (at 157.48 195.58 0)
+      (effects (font (size 1.27 1.27)) hide)
+    )
+    (property "DIGIKEY" "311-10.0KLRCT-ND" (at 157.48 195.58 0)
+      (effects (font (size 1.27 1.27)) hide)
+    )
     (pin "1")
     (pin "2")
@@
       (effects (font (size 1.27 1.27)) hide)
     )
+    (property "MPN" "RC0402FR-07330RL" (at 66.04 101.6 0)
+      (effects (font (size 1.27 1.27)) hide)
+    )
+    (property "MF" "Yageo" (at 66.04 101.6 0)
+      (effects (font (size 1.27 1.27)) hide)
+    )
+    (property "DIGIKEY" "311-330LRCT-ND" (at 66.04 101.6 0)
+      (effects (font (size 1.27 1.27)) hide)
+    )
