File: Hardware/KiCAD/Margay_1.kicad_sch (KiCad schematic)
At the start: 28 parts, among them J1 SDMMCWR-CRD, J4 USB_C, U1 ATMEGA1284M, U2 FT231X-Q

Commit message: KiCAD: populate MPN/MF/DIGIKEY fields from v3.0 BoM CSV
72 components updated with manufacturer, MPN, and DigiKey fields from
Margay_BoM_3v0_-_2023-03-17.csv. Fields were absent after Eagle→KiCAD
import. C20 (new 1µF DS3231M VCC decoupling cap) assigned same part as
C13/C14 (TMK107B7105KA-T). R22/R23 preserved as CRT0603-BY-1002ELF
(already correct). R7/R9 skipped — BoM MPN is a 330Ω part number, wrong
for the 1k value; needs manual correction.

Co-Authored-By: Claude Sonnet 4.6 <noreply@anthropic.com>
Parts:
- C1, C4, C5, C9: DIGIKEY (none) -> 490-4759-1-ND; MF (none) -> Murata; MPN (none) -> GCM155R71C104KA55D
- C2, C3: DIGIKEY (none) -> 490-12650-1-ND; MF (none) -> Murata; MPN (none) -> GCM1555C1H180JA16D
- C6: DIGIKEY (none) -> 490-6473-1-ND; MF (none) -> Murata; MPN (none) -> GRM21BR61C106KE15K
- C7, C8: DIGIKEY (none) -> 445-5585-1-ND; MF (none) -> TDK; MPN (none) -> CGA2B2C0G1H120J050BA
- H1, H2: DIGIKEY (none) -> DNP; MF (none) -> N/A; MPN (none) -> N/A
- J1: DIGIKEY (none) -> 732-3817-1-ND; MF (none) -> Wurth; MPN (none) -> 693063010911
- R1, R15, R16, R2: DIGIKEY (none) -> 311-10.0KLRCT-ND; MF (none) -> Yageo; MPN (none) -> RC0402FR-0710KL
- R3, R4: DIGIKEY (none) -> YAG3086CT-ND; MF (none) -> Yageo; MPN (none) -> RC0402FR-0727RL
- R31, R32: DIGIKEY (none) -> 311-5.10KLRCT-ND; MF (none) -> Yageo; MPN (none) -> RC0402FR-075K1L
- U1: DIGIKEY (none) -> ATMEGA1284P-MURCT-ND; MF (none) -> Atmel; MPN (none) -> ATMEGA1284P-MUR
- U2: DIGIKEY (none) -> 768-1128-1-ND; MF (none) -> FTDI; MPN (none) -> FT231XQ-R
Changed lines of the file:
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@@
+      (effects (font (size 1.27 1.27)) hide)
+    )
+    (property "MPN" "RC0402FR-0710KL" (at 68.58 137.16 0)
+      (effects (font (size 1.27 1.27)) hide)
+    )
+    (property "MF" "Yageo" (at 68.58 137.16 0)
+      (effects (font (size 1.27 1.27)) hide)
+    )
+    (property "DIGIKEY" "311-10.0KLRCT-ND" (at 68.58 137.16 0)
       (effects (font (size 1.27 1.27)) hide)
     )
@@
     )
     (property "Datasheet" "" (at 236.22 160.02 0)
+      (effects (font (size 1.27 1.27)) hide)
+    )
+    (property "MPN" "RC0402FR-0710KL" (at 236.22 160.02 0)
+      (effects (font (size 1.27 1.27)) hide)
+    )
+    (property "MF" "Yageo" (at 236.22 160.02 0)
+      (effects (font (size 1.27 1.27)) hide)
+    )
+    (property "DIGIKEY" "311-10.0KLRCT-ND" (at 236.22 160.02 0)
       (effects (font (size 1.27 1.27)) hide)
     )
@@
     )
     (property "Datasheet" "" (at 226.06 81.28 0)
+      (effects (font (size 1.27 1.27)) hide)
+    )
+    (property "MPN" "FT231XQ-R" (at 226.06 81.28 0)
+      (effects (font (size 1.27 1.27)) hide)
+    )
+    (property "MF" "FTDI" (at 226.06 81.28 0)
+      (effects (font (size 1.27 1.27)) hide)
+    )
+    (property "DIGIKEY" "768-1128-1-ND" (at 226.06 81.28 0)
       (effects (font (size 1.27 1.27)) hide)
     )
@@
       (effects (font (size 1.27 1.27)) hide)
     )
+    (property "MPN" "RC0402FR-0710KL" (at 226.06 152.4 0)
+      (effects (font (size 1.27 1.27)) hide)
+    )
+    (property "MF" "Yageo" (at 226.06 152.4 0)
+      (effects (font (size 1.27 1.27)) hide)
+    )
+    (property "DIGIKEY" "311-10.0KLRCT-ND" (at 226.06 152.4 0)
+      (effects (font (size 1.27 1.27)) hide)
+    )
     (pin "1")
     (pin "2")
@@
       (effects (font (size 1.27 1.27)) hide)
     )
+    (property "MPN" "GCM1555C1H180JA16D" (at 53.34 147.32 0)
+      (effects (font (size 1.27 1.27)) hide)
+    )
+    (property "MF" "Murata" (at 53.34 147.32 0)
+      (effects (font (size 1.27 1.27)) hide)
+    )
+    (property "DIGIKEY" "490-12650-1-ND" (at 53.34 147.32 0)
+      (effects (font (size 1.27 1.27)) hide)
+    )
     (pin "1")
     (pin "2")
@@
       (effects (font (size 1.27 1.27)) hide)
     )
+    (property "MPN" "GCM155R71C104KA55D" (at 180.34 40.64 0)
+      (effects (font (size 1.27 1.27)) hide)
+    )
+    (property "MF" "Murata" (at 180.34 40.64 0)
+      (effects (font (size 1.27 1.27)) hide)
+    )
+    (property "DIGIKEY" "490-4759-1-ND" (at 180.34 40.64 0)
+      (effects (font (size 1.27 1.27)) hide)
+    )
     (pin "1")
     (pin "2")
@@
       (effects (font (size 1.27 1.27)) hide)
     )
+    (property "MPN" "RC0402FR-075K1L" (at 157.48 58.42 0)
+      (effects (font (size 1.27 1.27)) hide)
+    )
+    (property "MF" "Yageo" (at 157.48 58.42 0)
+      (effects (font (size 1.27 1.27)) hide)
+    )
+    (property "DIGIKEY" "311-5.10KLRCT-ND" (at 157.48 58.42 0)
+      (effects (font (size 1.27 1.27)) hide)
+    )
     (pin "1")
     (pin "2")
@@
       (effects (font (size 1.27 1.27)) hide)
     )
+    (property "MPN" "RC0402FR-0710KL" (at 53.34 76.2 0)
+      (effects (font (size 1.27 1.27)) hide)
+    )
+    (property "MF" "Yageo" (at 53.34 76.2 0)
+      (effects (font (size 1.27 1.27)) hide)
+    )
+    (property "DIGIKEY" "311-10.0KLRCT-ND" (at 53.34 76.2 0)
+      (effects (font (size 1.27 1.27)) hide)
+    )
     (pin "1")
     (pin "2")
@@
     )
     (property "Datasheet" "" (at 101.6 172.72 0)
+      (effects (font (size 1.27 1.27)) hide)
+    )
+    (property "MPN" "ATMEGA1284P-MUR" (at 101.6 172.72 0)
+      (effects (font (size 1.27 1.27)) hide)
+    )
+    (property "MF" "Atmel" (at 101.6 172.72 0)
+      (effects (font (size 1.27 1.27)) hide)
+    )
+    (property "DIGIKEY" "ATMEGA1284P-MURCT-ND" (at 101.6 172.72 0)
       (effects (font (size 1.27 1.27)) hide)
     )
@@
       (effects (font (size 1.27 1.27)) hide)
     )
+    (property "MPN" "RC0402FR-075K1L" (at 167.64 58.42 0)
+      (effects (font (size 1.27 1.27)) hide)
+    )
+    (property "MF" "Yageo" (at 167.64 58.42 0)
+      (effects (font (size 1.27 1.27)) hide)
+    )
+    (property "DIGIKEY" "311-5.10KLRCT-ND" (at 167.64 58.42 0)
+      (effects (font (size 1.27 1.27)) hide)
+    )
     (pin "2")
     (pin "1")
@@
     )
     (property "Datasheet" "" (at 81.28 66.04 0)
+      (effects (font (size 1.27 1.27)) hide)
+    )
+    (property "MPN" "693063010911" (at 81.28 66.04 0)
+      (effects (font (size 1.27 1.27)) hide)
+    )
+    (property "MF" "Wurth" (at 81.28 66.04 0)
+      (effects (font (size 1.27 1.27)) hide)
+    )
+    (property "DIGIKEY" "732-3817-1-ND" (at 81.28 66.04 0)
       (effects (font (size 1.27 1.27)) hide)
     )
@@
       (effects (font (size 1.27 1.27)) hide)
     )
+    (property "MPN" "CGA2B2C0G1H120J050BA" (at 172.72 83.82 0)
+      (effects (font (size 1.27 1.27)) hide)
+    )
+    (property "MF" "TDK" (at 172.72 83.82 0)
+      (effects (font (size 1.27 1.27)) hide)
+    )
+    (property "DIGIKEY" "445-5585-1-ND" (at 172.72 83.82 0)
+      (effects (font (size 1.27 1.27)) hide)
+    )
     (pin "1")
     (pin "2")
@@
       (effects (font (size 1.27 1.27)) hide)
     )
+    (property "MPN" "N/A" (at 266.7 193.04 0)
+      (effects (font (size 1.27 1.27)) hide)
+    )
+    (property "MF" "N/A" (at 266.7 193.04 0)
+      (effects (font (size 1.27 1.27)) hide)
+    )
+    (property "DIGIKEY" "DNP" (at 266.7 193.04 0)
+      (effects (font (size 1.27 1.27)) hide)
+    )
     (instances
       (project "Margay"
@@
       (effects (font (size 1.27 1.27)) hide)
     )
+    (property "MPN" "RC0402FR-0727RL" (at 193.04 68.58 0)
+      (effects (font (size 1.27 1.27)) hide)
+    )
+    (property "MF" "Yageo" (at 193.04 68.58 0)
+      (effects (font (size 1.27 1.27)) hide)
+    )
+    (property "DIGIKEY" "YAG3086CT-ND" (at 193.04 68.58 0)
+      (effects (font (size 1.27 1.27)) hide)
+    )
     (pin "1")
     (pin "2")
@@
     )
     (property "Datasheet" "" (at 200.66 91.44 0)
+      (effects (font (size 1.27 1.27)) hide)
+    )
+    (property "MPN" "GCM155R71C104KA55D" (at 200.66 91.44 0)
+      (effects (font (size 1.27 1.27)) hide)
+    )
+    (property "MF" "Murata" (at 200.66 91.44 0)
+      (effects (font (size 1.27 1.27)) hide)
+    )
+    (property "DIGIKEY" "490-4759-1-ND" (at 200.66 91.44 0)
       (effects (font (size 1.27 1.27)) hide)
     )
@@
       (effects (font (size 1.27 1.27)) hide)
     )
+    (property "MPN" "N/A" (at 274.32 193.04 0)
+      (effects (font (size 1.27 1.27)) hide)
+    )
+    (property "MF" "N/A" (at 274.32 193.04 0)
+      (effects (font (size 1.27 1.27)) hide)
+    )
+    (property "DIGIKEY" "DNP" (at 274.32 193.04 0)
+      (effects (font (size 1.27 1.27)) hide)
+    )
     (instances
       (project "Margay"
@@
       (effects (font (size 1.27 1.27)) hide)
     )
+    (property "MPN" "RC0402FR-0727RL" (at 193.04 76.2 0)
+      (effects (font (size 1.27 1.27)) hide)
+    )
+    (property "MF" "Yageo" (at 193.04 76.2 0)
+      (effects (font (size 1.27 1.27)) hide)
+    )
+    (property "DIGIKEY" "YAG3086CT-ND" (at 193.04 76.2 0)
+      (effects (font (size 1.27 1.27)) hide)
+    )
     (pin "1")
     (pin "2")
@@
     )
     (property "Datasheet" "" (at 68.58 160.02 0)
+      (effects (font (size 1.27 1.27)) hide)
+    )
+    (property "MPN" "GCM155R71C104KA55D" (at 68.58 160.02 0)
+      (effects (font (size 1.27 1.27)) hide)
+    )
+    (property "MF" "Murata" (at 68.58 160.02 0)
+      (effects (font (size 1.27 1.27)) hide)
+    )
+    (property "DIGIKEY" "490-4759-1-ND" (at 68.58 160.02 0)
       (effects (font (size 1.27 1.27)) hide)
     )
@@
       (effects (font (size 1.27 1.27)) hide)
     )
+    (property "MPN" "GCM155R71C104KA55D" (at 53.34 134.62 0)
+      (effects (font (size 1.27 1.27)) hide)
+    )
+    (property "MF" "Murata" (at 53.34 134.62 0)
+      (effects (font (size 1.27 1.27)) hide)
+    )
+    (property "DIGIKEY" "490-4759-1-ND" (at 53.34 134.62 0)
+      (effects (font (size 1.27 1.27)) hide)
+    )
     (pin "1")
     (pin "2")
@@
       (effects (font (size 1.27 1.27)) hide)
     )
+    (property "MPN" "GCM1555C1H180JA16D" (at 53.34 152.4 0)
+      (effects (font (size 1.27 1.27)) hide)
+    )
+    (property "MF" "Murata" (at 53.34 152.4 0)
+      (effects (font (size 1.27 1.27)) hide)
+    )
+    (property "DIGIKEY" "490-12650-1-ND" (at 53.34 152.4 0)
+      (effects (font (size 1.27 1.27)) hide)
+    )
     (pin "1")
     (pin "2")
@@
       (effects (font (size 1.27 1.27)) hide)
     )
+    (property "MPN" "CGA2B2C0G1H120J050BA" (at 185.42 83.82 0)
+      (effects (font (size 1.27 1.27)) hide)
+    )
+    (property "MF" "TDK" (at 185.42 83.82 0)
+      (effects (font (size 1.27 1.27)) hide)
+    )
+    (property "DIGIKEY" "445-5585-1-ND" (at 185.42 83.82 0)
+      (effects (font (size 1.27 1.27)) hide)
+    )
     (pin "1")
     (pin "2")
@@
       (effects (font (size 1.27 1.27)) hide)
     )
+    (property "MPN" "GRM21BR61C106KE15K" (at 190.5 40.64 0)
+      (effects (font (size 1.27 1.27)) hide)
+    )
+    (property "MF" "Murata" (at 190.5 40.64 0)
+      (effects (font (size 1.27 1.27)) hide)
+    )
+    (property "DIGIKEY" "490-6473-1-ND" (at 190.5 40.64 0)
+      (effects (font (size 1.27 1.27)) hide)
+    )

Commit message: KiCAD: fix R7/R9 MPN (330Ω part number was wrong for 1k resistors)
The v3.0 BoM CSV had RC0603FR-07330RL (330Ω) as the MPN for R7 and R9,
but the DigiKey number and value were correct (1k). Boards were built
correctly. Updated MPN to RC0402FR-071KL to match the actual part.

Co-Authored-By: Claude Sonnet 4.6 <noreply@anthropic.com>
Parts:
- R7, R9: MPN RC0603FR-07330RL -> RC0402FR-071KL
Changed lines of the file:
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@@
       (effects (font (size 1.27 1.27)) hide)
     )
-    (property "MPN" "RC0603FR-07330RL" (at 261.62 66.04 90)
+    (property "MPN" "RC0402FR-071KL" (at 261.62 66.04 90)
       (effects (font (size 1.27 1.27)) (justify right top) hide)
     )
@@
       (effects (font (size 1.27 1.27)) hide)
     )
-    (property "MPN" "RC0603FR-07330RL" (at 271.78 71.12 90)
+    (property "MPN" "RC0402FR-071KL" (at 271.78 71.12 90)
       (effects (font (size 1.27 1.27)) (justify right top) hide)
     )
